Commit message: broader stack updated and integrate, odom, sensing in rviz, etc now runs. Next steps include testing (see the bottom of the readme), transforms for pole and bolts also now require integration. Documentation in the readme also required

File: rto4_description/urdf/rover/base.urdf.xacro (robot description, xacro)
@@ -1,11 +1,15 @@
 <?xml version="1.0"?>
 <robot name="robotino4_barebones_body" xmlns:xacro="http://www.ros.org/wiki/xacro">
+    <xacro:arg name="prefix" default=""/>
     <xacro:include filename="$(find rto4_description)/urdf/util/common_properties.xacro" />
+  <!-- ************************** Robotino4 Macro ***************************** -->
+  <xacro:macro name="robotino4" params="prefix:=''">
+    <xacro:property name="frame_ns" value="${prefix + '/' if prefix != '' else ''}" />
   <!-- *************************** Base Footprint ***************************** -->
-  <link name="base_footprint">
+  <link name="${frame_ns}base_footprint">
   </link>
   <!-- ************************************************************************ -->
   <!-- ****************************** Main Body ******************************* -->
-  <link name="base_link">
+  <link name="${frame_ns}base_link">
     <visual>
       <origin xyz="0 0 0.035" rpy="0 0 ${pi / 2}"/>
@@ -27,13 +31,13 @@
   </link>
   <!-- ========= Main Body - Joint ========= -->
-  <joint name="base_joint" type="fixed">
+  <joint name="${frame_ns}base_joint" type="fixed">
     <origin xyz="0 0 0" rpy="0 0 0"/>
-    <parent link="base_footprint"/>
-    <child link="base_link"/>
+    <parent link="${frame_ns}base_footprint"/>
+    <child link="${frame_ns}base_link"/>
   </joint>
   <!-- ************************************************************************ -->
   <!-- ***************************** Wheel Macro ****************************** -->
-  <xacro:macro name="wheel_link" params="number">
-    <link name="wheel${number}_link">
+  <xacro:macro name="wheel_link" params="prefix_ns number">
+    <link name="${prefix_ns}wheel${number}_link">
       <visual>
         <origin xyz="0 0 0" rpy="0 0 0"/>
@@ -55,28 +59,40 @@
     </link>
   </xacro:macro>
-  <xacro:wheel_link number="0" />
-  <xacro:wheel_link number="1" />
-  <xacro:wheel_link number="2" />
+  <xacro:wheel_link prefix_ns="${frame_ns}" number="0" />
+  <xacro:wheel_link prefix_ns="${frame_ns}" number="1" />
+  <xacro:wheel_link prefix_ns="${frame_ns}" number="2" />
   <!-- ========== Wheel 0 - Joint ========== -->
-  <joint name="wheel0_joint" type="fixed">   <!--<joint name="wheel0_joint" type="continuous"></joint> -->
-    <parent link="base_link"/>
-    <child link="wheel0_link"/>
+  <joint name="${frame_ns}wheel0_joint" type="fixed">   <!--<joint name="wheel0_joint" type="continuous"></joint> -->
+    <parent link="${frame_ns}base_link"/>
+    <child link="${frame_ns}wheel0_link"/>
     <origin xyz="-0.1825 -0.0001 0.059154" rpy="0 0 ${pi / 2}"/>
     <axis xyz="0 1 0" rpy="0 0 0"/>
   </joint>
   <!-- ========== Wheel 1 - Joint ========== -->
-  <joint name="wheel1_joint" type="fixed">
-    <parent link="base_link"/>
-    <child link="wheel1_link"/>
+  <joint name="${frame_ns}wheel1_joint" type="fixed">
+    <parent link="${frame_ns}base_link"/>
+    <child link="${frame_ns}wheel1_link"/>
     <origin xyz="0.090625 -0.157067 0.059154" rpy="0 0 ${(30 * (pi/2)) / 90}"/>
     <axis xyz="0 1 0" rpy="0 0 0"/>
   </joint>
   <!-- ========== Wheel 2 - Joint ========== -->
-  <joint name="wheel2_joint" type="fixed">
-    <parent link="base_link"/>
-    <child link="wheel2_link"/>
+  <joint name="${frame_ns}wheel2_joint" type="fixed">
+    <parent link="${frame_ns}base_link"/>
+    <child link="${frame_ns}wheel2_link"/>
     <origin xyz="0.090625 0.156867 0.059154" rpy="0 0 ${-(30 * (pi/2)) / 90}"/>
     <axis xyz="0 1 0" rpy="0 0 0"/>
   </joint>
   <!-- ************************************************************************ -->
+  <!-- ****************************** Laser Link ****************************** -->
+  <link name="${frame_ns}laser_link">
+  </link>
+  <joint name="${frame_ns}laser_joint" type="fixed">
+    <parent link="${frame_ns}base_link"/>
+    <child link="${frame_ns}laser_link"/>
+    <origin xyz="0 0 0.14" rpy="0 0 0"/>
+  </joint>
+  <!-- ************************************************************************ -->
+  </xacro:macro>
+  <!-- Default instantiation for standalone use -->
+  <xacro:robotino4 prefix="$(arg prefix)" />
 </robot>
